Commit message: turn falcon_base to intrinsic frame in world

File: urdf/floating_grip.urdf.xacro (robot description, xacro)
@@ -38,5 +38,5 @@
   <parent link="world"/>
   <child link="falcon_base"/>
-  <origin xyz="0 0 0" rpy="${tau/4} 0 0"/>
+  <origin xyz="0 0 0" rpy="${tau/4} 0 ${tau/4}"/>
 </joint>
 </robot>

Commit message: changed to use macro
separated in a standalone and macro to use in a diffrent urdf

File: urdf/floating_grip.urdf.xacro (robot description, xacro)
@@ -1,4 +1,5 @@
 <robot name="floating_gripper" xmlns:xacro="http://www.ros.org/wiki/xacro" xmlns:falcon_ros="http://www.falcon-ros.org">
 <!-- TODO: the mesh geometries here do not make much sense yet, but appears sufficient at first glance -->
+<xacro:macro name="falcon">
 <link name="falcon_base">
   <visual>
@@ -34,9 +35,4 @@
   <origin xyz="0 0 0.0" rpy="0 0 0"/>
 </joint>
-<link name="world"/>
-<joint name="world_joint" type="fixed">
-  <parent link="world"/>
-  <child link="falcon_base"/>
-  <origin xyz="0 0 0" rpy="${tau/4} 0 ${tau/4}"/>
-</joint>
+</xacro:macro>
 </robot>
